File: MeterBoard32.sch (KiCad schematic (older format))
At the start: 33 parts, among them J1 Screw_Terminal_01x02, M1 MICRO_USB_18_TH, Q1 S8050, Q2 S8050, U1 AMS1117-3V3, U2 CP2102N-GQFN24, U3 ESP32-WROOM, U4 TSS721A

Commit message: Added schematics for TSS721A
Parts:
- added C?: C_Small, symbol C_Small
- added R?: 100, symbol R_Small
Connections:
- wire segments 103 -> 107
Other:
- moved on the sheet: R?
