File: MeterBoard32.sch (KiCad schematic (older format))
At the start: 36 parts, among them J1 Screw_Terminal_01x02, M1 MICRO_USB_18_TH, Q1 S8050, Q2 S8050, U1 AMS1117-3V3, U2 CP2102N-GQFN24, U3 ESP32-WROOM, U5 TSS721A

Commit message: Fixed 3D models
Parts:
- Q1, Q2: symbol Transistor_BJT:S8050 -> MeterBoard32-rescue:S8050-Transistor_BJT
Changed lines of the file:
@@
 RTS
 $Comp
-L Transistor_BJT:S8050 Q1
+L MeterBoard32-rescue:S8050-Transistor_BJT Q1
 U 1 1 5AAAA0A6
 P 7050 4100
@@
 	1700 4500 1700 4550
 $Comp
-L Transistor_BJT:S8050 Q2
+L MeterBoard32-rescue:S8050-Transistor_BJT Q2
 U 1 1 5AAAA111
 P 7050 4650

Commit message: Finished the conversion of MeterBoard32 from KiCad 4 to KiCad 5
Parts:
- Q1, Q2: symbol MeterBoard32-rescue:S8050-Transistor_BJT -> Transistor_BJT:2N3055
Other:
- moved on the sheet: C7, D1, D5
Changed lines of the file:
@@
 Sheet 1 1
 Title "MeterBoard32"
-Date "2021-04-26"
+Date "2021-04-27"
 Rev "2"
 Comp "Henrik Nelson"
@@
 Text Label 6400 4100 2    60   ~ 0
 DTR
-Text Label 6400 4650 2    60   ~ 0
+Text Label 6350 4650 2    60   ~ 0
 RTS
 $Comp
-L MeterBoard32-rescue:S8050-Transistor_BJT Q1
+L Transistor_BJT:2N3055 Q1
 U 1 1 5AAAA0A6
 P 7050 4100
@@
 L LED:WS2812B D5
 U 1 1 5AAACD5F
-P 4750 4200
-F 0 "D5" V 4527 4406 50  0000 R BNN
-F 1 "WS2812B" V 4965 3821 50  0000 L TNN
-F 2 "LED_SMD:LED_WS2812B_PLCC4_5.0x5.0mm_P3.2mm" H 4800 3900 50  0001 L TNN
-F 3 "" H 4850 3825 50  0001 L TNN
-	1    4750 4200
+P 4700 4200
+F 0 "D5" V 4477 4406 50  0000 R BNN
+F 1 "WS2812B" V 4915 3821 50  0000 L TNN
+F 2 "LED_SMD:LED_WS2812B_PLCC4_5.0x5.0mm_P3.2mm" H 4750 3900 50  0001 L TNN
+F 3 "" H 4800 3825 50  0001 L TNN
+	1    4700 4200
 	0    -1   -1   0
 $EndComp
@@
 L Device:C_Small C7
 U 1 1 5AAADC04
-P 4750 4700
-F 0 "C7" V 4650 4650 50  0000 L CNN
-F 1 "0.1uF" V 4850 4600 50  0000 L CNN
-F 2 "Capacitor_SMD:C_1206_3216Metric_Pad1.33x1.80mm_HandSolder" H 4750 4700 50  0001 C CNN
-F 3 "" H 4750 4700 50  0001 C CNN
-	1    4750 4700
+P 4700 4700
+F 0 "C7" V 4600 4650 50  0000 L CNN
+F 1 "0.1uF" V 4800 4600 50  0000 L CNN
+F 2 "Capacitor_SMD:C_1206_3216Metric_Pad1.33x1.80mm_HandSolder" H 4700 4700 50  0001 C CNN
+F 3 "" H 4700 4700 50  0001 C CNN
+	1    4700 4700
 	0    1    1    0
 $EndComp
@@
 L power:GND #PWR014
 U 1 1 5AAAE073
-P 5150 4450
-F 0 "#PWR014" H 5150 4200 50  0001 C CNN
-F 1 "GND" H 5150 4300 50  0000 C CNN
-F 2 "" H 5150 4450 50  0001 C CNN
-F 3 "" H 5150 4450 50  0001 C CNN
-	1    5150 4450
+P 5100 4700
+F 0 "#PWR014" H 5100 4450 50  0001 C CNN
+F 1 "GND" H 5100 4550 50  0000 C CNN
+F 2 "" H 5100 4700 50  0001 C CNN
+F 3 "" H 5100 4700 50  0001 C CNN
+	1    5100 4700
 	0    -1   -1   0
 $EndComp
@@
 L power:VBUS #PWR015
 U 1 1 5AAAE0B7
-P 4350 4450
-F 0 "#PWR015" H 4350 4300 50  0001 C CNN
-F 1 "VBUS" H 4350 4600 50  0000 C CNN
-F 2 "" H 4350 4450 50  0001 C CNN
-F 3 "" H 4350 4450 50  0001 C CNN
-	1    4350 4450
+P 4300 4700
+F 0 "#PWR015" H 4300 4550 50  0001 C CNN
+F 1 "VBUS" H 4300 4850 50  0000 C CNN
+F 2 "" H 4300 4700 50  0001 C CNN
+F 3 "" H 4300 4700 50  0001 C CNN
+	1    4300 4700
 	0    -1   -1   0
 $EndComp
@@
 	1    0    0    -1
 $EndComp
-NoConn ~ 4750 3900
+NoConn ~ 4700 3900
 $Comp
 L Regulator_Linear:AMS1117-3.3 U1
@@
 	7150 4350 6450 4350
 Wire Wire Line
-	6400 4650 6450 4650
+	6350 4650 6450 4650
 Wire Wire Line
 	6750 4650 6850 4650
@@
 Wire Notes Line
 	8500 5000 8500 3700
-Wire Wire Line
-	5150 4200 5150 4450
 Wire Notes Line
 	5450 600  8400 600
@@
 	2900 3150 3100 3150
 Wire Wire Line
-	4450 4200 4350 4200
-Wire Wire Line
-	5150 4700 5150 4450
-Connection ~ 5150 4450
-Wire Wire Line
-	4350 4200 4350 4450
-Wire Wire Line
-	4650 4700 4350 4700
-Connection ~ 4350 4450
-Wire Wire Line
-	4350 4700 4350 4450
+	4400 4200 4350 4200
+Wire Wire Line
+	4350 4200 4350 4700
+Wire Wire Line
+	4600 4700 4350 4700
 Wire Wire Line
 	1700 4550 2150 4550
@@
 	2000 4200 2150 4200
 Wire Wire Line
-	4850 4700 5150 4700
-Wire Wire Line
-	5150 4200 5050 4200
+	4800 4700 5050 4700
 Wire Wire Line
 	6100 1100 6100 1550
@@
 	1250 2250 1350 2250
 Wire Wire Line
-	1400 1850 1250 1850
+	1350 1850 1250 1850
 Wire Notes Line
 	600  3550 600  600
@@
 L Diode:1N5819 D1
 U 1 1 5AB03155
-P 1550 1850
-F 0 "D1" H 1550 1950 50  0000 C CNN
-F 1 "1N5819/SS14" H 1550 1750 50  0000 C CNN
-F 2 "Diode_SMD:D_SOD-123F" H 1550 1675 50  0001 C CNN
-F 3 "" H 1550 1850 50  0001 C CNN
-	1    1550 1850
+P 1500 1850
+F 0 "D1" H 1500 1950 50  0000 C CNN
+F 1 "1N5819/SS14" H 1500 1750 50  0000 C CNN
+F 2 "Diode_SMD:D_SOD-123F" H 1500 1675 50  0001 C CNN
+F 3 "" H 1500 1850 50  0001 C CNN
+	1    1500 1850
 	-1   0    0    1
 $EndComp
@@
 	1250 2050 1300 2050
 Wire Wire Line
-	1700 1850 1900 1850
+	1650 1850 1900 1850
 Wire Wire Line
 	1350 2250 1350 2300
@@
 	1700 4500 1700 4550
 $Comp
-L MeterBoard32-rescue:S8050-Transistor_BJT Q2
+L Transistor_BJT:2N3055 Q2
 U 1 1 5AAAA111
 P 7050 4650
@@
 	1    0    0    1
 $EndComp
+Connection ~ 4350 4700
+Wire Wire Line
+	4350 4700 4300 4700
+Wire Wire Line
+	5000 4200 5050 4200
+Wire Wire Line
+	5050 4200 5050 4700
+Connection ~ 5050 4700
+Wire Wire Line
+	5050 4700 5100 4700
+Wire Wire Line
+	4700 4500 4750 4500
 $EndSCHEMATC
